File: IoT/Oblig1/tinker_cad_board.brd (EAGLE design)
At the start: 68.6 x 53.3 mm, 10 parts

Commit message: Finished assignment
Parts:
- added R4, R5: 10k‎Ω, AUTODESK_CIRCUITS_BREADBOARD:0207/10
Connections:
- removed net N$12 (its old number): PIR1.1, R1.1, R2.1, R3.1, S1.4, S2.4, U1.GND..
- new net N$15: PIR1.2, S1.4, S2.4, U1.5V
- net N$10: now also U1.5; no longer U1.7
- net N$11: now also PIR1.1, R1.1, R2.1, R3.1, R4.1, R5.1, U1.GND..; no longer PIR1.2, U1.5V
- net N$2: now also U1.3; no longer U1.4
- net N$3: now also R5.2
- net N$6: now also R4.2
